File: PCB/Artnet_DMX_Converter/Microcontroller.kicad_sch (KiCad schematic)
At the start: 37 parts, among them J1 Conn_01x03_MountingPin, SW1 SW_Push, SW2 SW_Push, U1 RP2350B, U2 W25Q128JVS, Y1 ABM8-272-T3

Commit message: Fixed RP2350 power layout
Parts:
- C15, C16: footprint Capacitor_SMD:C_0402_1005Metric -> RP2350_80QFN_minimal:C_0402_1005Metric_small_pads
- L1: footprint LCSC:IND-SMD_L2.0-W1.6_AOTA-B201610S3R3-101-T -> RP2350_80QFN_minimal:L_pol_2016
- U1: footprint Package_DFN_QFN:QFN-80-1EP_10x10mm_P0.4mm_EP3.4x3.4mm -> RP2350_80QFN_minimal:RP2350-QFN-80-1EP_10x10_P0.4mm_EP3.4x3.4mm_ThermalVias
Changed lines of the file:
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@@
 			)
 		)
-		(property "Footprint" "LCSC:IND-SMD_L2.0-W1.6_AOTA-B201610S3R3-101-T"
+		(property "Footprint" "RP2350_80QFN_minimal:L_pol_2016"
 			(at 57.15 60.96 0)
 			(effects
@@
 			)
 		)
-		(property "Footprint" "Capacitor_SMD:C_0402_1005Metric"
+		(property "Footprint" "RP2350_80QFN_minimal:C_0402_1005Metric_small_pads"
 			(at 45.4152 66.04 0)
 			(effects
@@
 			)
 		)
-		(property "Footprint" "Package_DFN_QFN:QFN-80-1EP_10x10mm_P0.4mm_EP3.4x3.4mm"
+		(property "Footprint" "RP2350_80QFN_minimal:RP2350-QFN-80-1EP_10x10_P0.4mm_EP3.4x3.4mm_ThermalVias"
 			(at 146.05 97.79 0)
 			(effects
@@
 			)
 		)
-		(property "Footprint" "Capacitor_SMD:C_0402_1005Metric"
+		(property "Footprint" "RP2350_80QFN_minimal:C_0402_1005Metric_small_pads"
 			(at 32.7152 66.04 0)
 			(effects
